Commit message: v0.0.5

File: arm_description/urdf/arm.urdf.xacro (robot description, xacro)
@@ -1,7 +1,10 @@
 <?xml version="1.0"?>
 <robot name="robotarm" xmlns:xacro="http://www.ros.org/wiki/xacro">
+    <!-- materials -->
+    <material name="grey"><color rgba="0.5 0.5 0.5 1.0"/></material>
+    <material name="blue"><color rgba="0.1 0.1 0.8 1.0"/></material>
+    <material name="black"><color rgba="0.1 0.1 0.1 1.0"/></material>
     <xacro:include filename="arm_core.xacro" />
     <xacro:include filename="camera.xacro" />
-    <xacro:include filename="arm_gazebo.xacro" />
     <xacro:include filename="arm_control.xacro" />
 </robot>

File: arm_description/urdf/arm_control.xacro (robot description, xacro)
@@ -1,7 +1,7 @@
 <?xml version="1.0"?>
-<robot name="robotarm" xmlns:xacro="http://www.ros.org/wiki/xacro">
+<robot xmlns:xacro="http://www.ros.org/wiki/xacro">
     <ros2_control name="GazeboSystem" type="system">
         <hardware>
-            <plugin>gz_ros2_control/GzSystem</plugin>
+            <plugin>gz_ros2_control/GazeboSimSystem</plugin>
         </hardware>
         <joint name="joint_1">

File: arm_description/urdf/arm_core.xacro (robot description, xacro)
@@ -1,72 +1,153 @@
 <?xml version="1.0"?>
-<robot name="robotarm" xmlns:xacro="http://www.ros.org/wiki/xacro">
-    <material name="grey">
-      <color rgba="0.5 0.5 0.5 1.0"/>
-    </material>
-    <material name="blue">
-      <color rgba="0.1 0.1 0.8 1.0"/>
-    </material>
-    <material name="black">
-      <color rgba="0.1 0.1 0.1 1.0"/>
-    </material>
-    <xacro:property name="mesh_prefix" value="package://arm_description/meshes"/>
-    <xacro:property name="limit_lower" value="-1.54"/>
-    <xacro:property name="limit_upper" value="1.54"/>
-    <xacro:property name="limit_effort" value="100"/>
-    <xacro:property name="inertia_val" value="0.0001"/>
-    <xacro:macro name="arm_link_macro" params="link_name mass_val">
-        <link name="${link_name}">
-            <inertial>
-                <mass value="${mass_val}"/>
-                <inertia ixx="${inertia_val}" iyy="${inertia_val}" izz="${inertia_val}"/>
-            </inertial>
-            <visual>
-                <geometry><mesh filename="${mesh_prefix}/${link_name}.stl"/></geometry>
-            </visual>
-            <collision>
-                <geometry><mesh filename="${mesh_prefix}/${link_name}.stl"/></geometry>
-            </collision>
-        </link>
-    </xacro:macro>
-    <xacro:macro name="arm_joint_macro" params="joint_name parent_link child_link xyz axis_xyz">
-        <joint name="${joint_name}" type="revolute">
-            <parent link="${parent_link}"/>
-            <child link="${child_link}"/>
-            <origin xyz="${xyz}" rpy="0 0 0"/>
-            <axis xyz="${axis_xyz}"/>
-            <limit lower="${limit_lower}" upper="${limit_upper}" effort="${limit_effort}"/>
-        </joint>
-    </xacro:macro>
-    <link name='base_link'>
-        <inertial>
-            <mass value="0.5"/>
-            <inertia ixx="0.001" iyy="0.001" izz="0.001"/>
-        </inertial>
-        <visual>
-            <geometry><mesh filename="${mesh_prefix}/base_link.stl"/></geometry>
-            <material name="grey"/>
-        </visual>
-        <collision>
-            <geometry><mesh filename="${mesh_prefix}/base_link.stl"/></geometry>
-        </collision>
-    </link>
-    <xacro:arm_link_macro  link_name="link_1" mass_val="0.2"/>
-    <xacro:arm_joint_macro joint_name="joint_1" parent_link="base_link" child_link="link_1" xyz="0 0 0.0814" axis_xyz="0 0 1"/>
-    <xacro:arm_link_macro  link_name="link_2" mass_val="0.2"/>
-    <xacro:arm_joint_macro joint_name="joint_2" parent_link="link_1" child_link="link_2" xyz="-0.02 0 0.015" axis_xyz="0 -1 0"/>
-    <xacro:arm_link_macro  link_name="link_3" mass_val="0.2"/>
-    <xacro:arm_joint_macro joint_name="joint_3" parent_link="link_2" child_link="link_3" xyz="-0.0021 0 0.1035" axis_xyz="0 1 0"/>
-    <xacro:arm_link_macro  link_name="link_4" mass_val="0.1"/>
-    <xacro:arm_joint_macro joint_name="joint_4" parent_link="link_3" child_link="link_4" xyz="-0.002 0 0.1275" axis_xyz="0 -1 0"/>
-    <link name="tool_tip">
-      <inertial>
-        <mass value="0.01"/>
-        <inertia ixx="1e-6" ixy="0" ixz="0" iyy="1e-6" iyz="0" izz="1e-6"/>
-      </inertial>
-    </link>
-    <joint name="joint_tool" type="fixed">
-      <parent link="link_4"/>
-      <child link="tool_tip"/>
-      <origin xyz="0.01 0 0.092" rpy="0 0.0 0"/>
-    </joint>
+<robot xmlns:xacro="http://www.ros.org/wiki/xacro">
+  <!-- properties -->
+  <xacro:property name="mesh_prefix" value="package://arm_description/meshes"/>
+  <xacro:property name="limit_lower" value="-1.54"/>
+  <xacro:property name="limit_upper" value="1.54"/>
+  <xacro:property name="limit_effort" value="100"/>
+  <xacro:property name="limit_velocity" value="3.14"/>
+  <xacro:property name="inertia_val" value="0.0001"/>
+  <!-- ===================================================== -->
+  <!-- ==================== LINKS ======================== -->
+  <!-- ===================================================== -->
+  <!-- Base Link -->
+  <link name="base_link">
+    <inertial>
+      <origin xyz="0 0 0" rpy="0 0 0"/>
+      <mass value="0.5"/>
+      <inertia ixx="0.001" ixy="0.0" ixz="0.0" iyy="0.001" iyz="0.0" izz="0.001"/>
+    </inertial>
+    <visual>
+      <geometry><mesh filename="${mesh_prefix}/base_link.stl"/></geometry>
+      <material name="grey"/>
+    </visual>
+    <collision>
+      <geometry><box size="0.1 0.1 0.08"/></geometry>
+      <origin xyz="0 0 0.04" rpy="0 0 0"/>
+    </collision>
+  </link>
+  <!-- Link 1 -->
+  <link name="link_1">
+    <inertial>
+      <origin xyz="0 0 0" rpy="0 0 0"/>
+      <mass value="0.2"/>
+      <inertia ixx="${inertia_val}" ixy="0.0" ixz="0.0" iyy="${inertia_val}" iyz="0.0" izz="${inertia_val}"/>
+    </inertial>
+    <visual>
+      <geometry><mesh filename="${mesh_prefix}/link_1.stl"/></geometry>
+      <material name="blue"/>
+    </visual>
+    <collision>
+      <geometry><cylinder radius="0.02" length="0.1"/></geometry>
+      <origin xyz="0 0 0.05" rpy="0 0 0"/>
+    </collision>
+  </link>
+  <!-- Link 2 -->
+  <link name="link_2">
+    <inertial>
+      <origin xyz="0 0 0" rpy="0 0 0"/>
+      <mass value="0.2"/>
+      <inertia ixx="${inertia_val}" ixy="0.0" ixz="0.0" iyy="${inertia_val}" iyz="0.0" izz="${inertia_val}"/>
+    </inertial>
+    <visual>
+      <geometry><mesh filename="${mesh_prefix}/link_2.stl"/></geometry>
+      <material name="blue"/>
+    </visual>
+    <collision>
+      <geometry><cylinder radius="0.02" length="0.12"/></geometry>
+      <origin xyz="0 0 0.06" rpy="0 0 0"/>
+    </collision>
+  </link>
+  <!-- Link 3 -->
+  <link name="link_3">
+    <inertial>
+      <origin xyz="0 0 0" rpy="0 0 0"/>
+      <mass value="0.2"/>
+      <inertia ixx="${inertia_val}" ixy="0.0" ixz="0.0" iyy="${inertia_val}" iyz="0.0" izz="${inertia_val}"/>
+    </inertial>
+    <visual>
+      <geometry><mesh filename="${mesh_prefix}/link_3.stl"/></geometry>
+      <material name="blue"/>
+    </visual>
+    <collision>
+      <geometry><cylinder radius="0.02" length="0.12"/></geometry>
+      <origin xyz="0 0 0.06" rpy="0 0 0"/>
+    </collision>
+  </link>
+  <!-- Link 4 -->
+  <link name="link_4">
+    <inertial>
+      <origin xyz="0 0 0" rpy="0 0 0"/>
+      <mass value="0.1"/>
+      <inertia ixx="${inertia_val}" ixy="0.0" ixz="0.0" iyy="${inertia_val}" iyz="0.0" izz="${inertia_val}"/>
+    </inertial>
+    <visual>
+      <geometry><mesh filename="${mesh_prefix}/link_4.stl"/></geometry>
+      <material name="blue"/>
+    </visual>
+    <collision>
+      <geometry><cylinder radius="0.02" length="0.1"/></geometry>
+      <origin xyz="0 0 0.05" rpy="0 0 0"/>
+    </collision>
+  </link>
+  <!-- Tooltip Link -->
+  <link name="tool_tip">
+    <inertial>
+      <origin xyz="0 0 0" rpy="0 0 0"/>
+      <mass value="0.01"/>
+      <inertia ixx="1e-6" ixy="0.0" ixz="0.0" iyy="1e-6" iyz="0.0" izz="1e-6"/>
+    </inertial>
+  </link>
+  <!-- ===================================================== -->
+  <!-- ==================== JOINTS ======================= -->
+  <!-- ===================================================== -->
+  <!-- World Joint -->
+  <link name="world"/>
+  <joint name="world_to_base_joint" type="fixed">
+    <parent link="world"/>
+    <child link="base_link"/>
+    <origin xyz="0 0 0.002" rpy="0 0 0"/>
+  </joint>
+  <!-- Joint 1 -->
+  <joint name="joint_1" type="revolute">
+    <parent link="base_link"/>
+    <child link="link_1"/>
+    <origin xyz="0 0 0.0814" rpy="0 0 0"/>
+    <axis xyz="0 0 1"/>
+    <limit lower="${limit_lower}" upper="${limit_upper}" effort="${limit_effort}" velocity="${limit_velocity}"/>
+    <dynamics damping="0.7" friction="0.1"/>
+  </joint>
+  <!-- Joint 2 -->
+  <joint name="joint_2" type="revolute">
+    <parent link="link_1"/>
+    <child link="link_2"/>
+    <origin xyz="-0.02 0 0.015" rpy="0 0 0"/>
+    <axis xyz="0 -1 0"/>
+    <limit lower="${limit_lower}" upper="${limit_upper}" effort="${limit_effort}" velocity="${limit_velocity}"/>
+    <dynamics damping="0.7" friction="0.1"/>
+  </joint>
+  <!-- Joint 3 -->
+  <joint name="joint_3" type="revolute">
+    <parent link="link_2"/>
+    <child link="link_3"/>
+    <origin xyz="-0.0021 0 0.1035" rpy="0 0 0"/>
+    <axis xyz="0 1 0"/>
+    <limit lower="${limit_lower}" upper="${limit_upper}" effort="${limit_effort}" velocity="${limit_velocity}"/>
+    <dynamics damping="0.7" friction="0.1"/>
+  </joint>
+  <!-- Joint 4 -->
+  <joint name="joint_4" type="revolute">
+    <parent link="link_3"/>
+    <child link="link_4"/>
+    <origin xyz="-0.002 0 0.1275" rpy="0 0 0"/>
+    <axis xyz="0 -1 0"/>
+    <limit lower="${limit_lower}" upper="${limit_upper}" effort="${limit_effort}" velocity="${limit_velocity}"/>
+    <dynamics damping="0.7" friction="0.1"/>
+  </joint>
+  <!-- Tooltip Joint -->
+  <joint name="joint_tool" type="fixed">
+    <parent link="link_4"/>
+    <child link="tool_tip"/>
+    <origin xyz="0.01 0 0.092" rpy="0 0 0"/>
+  </joint>
 </robot>

File: arm_description/urdf/arm_gazebo.xacro (robot description, xacro)
@@ -1,8 +1,10 @@
 <?xml version="1.0"?>
-<robot name="robotarm" xmlns:xacro="http://www.ros.org/wiki/xacro">
+<robot xmlns:xacro="http://www.ros.org/wiki/xacro">
     <gazebo>
-        <plugin filename="gz-sim-joint-state-publisher-system"
-                name="gz::sim::systems::JointStatePublisher">
-            <topic>joint_states</topic>
+        <plugin filename="libgz_ros2_control-system.so" name="gz_ros2_control::GazeboSimROS2ControlPlugin">
+            <ros>
+                <namespace>/controller_manager</namespace>
+            </ros>
+            <parameters>$(find arm_gazebo)/params/arm_controllers.yaml</parameters>
         </plugin>
     </gazebo>

File: arm_description/urdf/camera.xacro (robot description, xacro)
@@ -1,48 +1,48 @@
 <?xml version="1.0"?>
-<robot name="robotarm" xmlns:xacro="http://www.ros.org/wiki/xacro">
-    <link name='camera_link'>
-        <visual><geometry><mesh filename="package://arm_description/meshes/camera.stl"/></geometry></visual>
-        <collision><geometry><mesh filename="package://arm_description/meshes/camera.stl"/></geometry></collision>
-        <inertial>
-            <mass value="0.05"/>
-            <inertia ixx="1e-6" iyy="1e-6" izz="1e-6"/>
-        </inertial>
-    </link>
-    <link name="camera_optical_frame"/>
-    <joint name='camera_joint' type='fixed'>
-        <parent link='link_4'/>
-        <child link='camera_link'/>
-        <origin xyz="-0.0035 0 0.054" rpy="0 0 0"/>
-    </joint>
-    <joint name="camera_optical_joint" type="fixed">
-        <parent link="camera_link"/>
-        <child link="camera_optical_frame"/>
-        <origin xyz="0 0 0.01" rpy="${-pi/2} 0 ${-pi/2}"/>
-    </joint>
-    <gazebo reference="camera_optical_frame">
-        <sensor type="camera" name="my_camera">
-            <update_rate>30.0</update_rate>
-            <camera name="head">
-                <horizontal_fov>1.0466</horizontal_fov>
-                <image>
-                    <width>800</width>
-                    <height>600</height>
-                    <format>R8G8B8</format>
-                </image>
-                <clip>
-                    <near>0.02</near>
-                    <far>300</far>
-                </clip>
-                <distortion>
-                    <k1>-0.414921465</k1>
-                    <k2>0.277976117</k2>
-                    <p1>0.000362302582</p1>
-                    <p2>-0.000173492775</p2>
-                    <k3>-0.194112104</k3>
-                    <center>0.5 0.5</center>
-                </distortion>
-            </camera>
-            <plugin filename="libgz-sim-ros2-camera-system.so" name="gz::sim::systems::Ros2Camera"/>
-        </sensor>
-    </gazebo>
+<robot xmlns:xacro="http://www.ros.org/wiki/xacro">
+  <link name='camera_link'>
+    <visual>
+      <geometry><mesh filename="package://arm_description/meshes/camera.stl"/></geometry><material name="black"/>
+    </visual>
+    <collision>
+      <geometry><box size="0.02 0.04 0.03"/></geometry>
+    </collision>
+    <!-- inertial: 6성분 모두 명시 (비대각은 0으로 안전) -->
+    <inertial>
+      <origin xyz="0 0 0" rpy="0 0 0"/>
+      <mass value="0.05"/>
+      <inertia
+        ixx="1e-6" ixy="0.0" ixz="0.0"
+        iyy="1e-6" iyz="0.0"
+        izz="1e-6"/>
+    </inertial>
+  </link>
+  <link name="camera_optical_frame"/>
+  <joint name='camera_joint' type='fixed'>
+    <parent link='link_4'/>
+    <child link='camera_link'/>
+    <origin xyz="-0.0035 0 0.054" rpy="0 0 0"/>
+  </joint>
+  <joint name="camera_optical_joint" type="fixed">
+    <parent link="camera_link"/>
+    <child link="camera_optical_frame"/>
+    <origin rpy="0 0 -1.57079632679" xyz="0 0 0.01"/>
+  </joint>
+  <gazebo reference="camera_optical_frame">
+    <sensor type="camera" name="my_camera">
+      <topic>/camera/image_raw</topic>
+      <update_rate>30.0</update_rate>
+      <camera name="head">
+        <horizontal_fov>1.0466</horizontal_fov>
+        <image><width>800</width><height>600</height><format>R8G8B8</format></image>
+        <clip><near>0.02</near><far>300</far></clip>
+        <distortion>
+          <k1>-0.414921465</k1><k2>0.277976117</k2>
+          <p1>0.000362302582</p1><p2>-0.000173492775</p2>
+          <k3>-0.194112104</k3>
+          <center>0.5 0.5</center>
+        </distortion>
+      </camera>
+    </sensor>
+  </gazebo>
 </robot>

Commit message: v.0.0.6

File: arm_description/urdf/arm.urdf.xacro (robot description, xacro)
@@ -8,3 +8,4 @@
     <xacro:include filename="camera.xacro" />
     <xacro:include filename="arm_control.xacro" />
+    <xacro:include filename="arm_gazebo.xacro" />
 </robot>

File: arm_description/urdf/arm_control.xacro (robot description, xacro)
@@ -1,5 +1,5 @@
 <?xml version="1.0"?>
 <robot xmlns:xacro="http://www.ros.org/wiki/xacro">
-    <ros2_control name="GazeboSystem" type="system">
+    <ros2_control name="GazeboSimSystem" type="system">
         <hardware>
             <plugin>gz_ros2_control/GazeboSimSystem</plugin>

File: arm_description/urdf/arm_gazebo.xacro (robot description, xacro)
@@ -3,8 +3,8 @@
     <gazebo>
         <plugin filename="libgz_ros2_control-system.so" name="gz_ros2_control::GazeboSimROS2ControlPlugin">
+            <parameters>$(find arm_gazebo)/params/arm_controllers.yaml</parameters>
             <ros>
-                <namespace>/controller_manager</namespace>
+                <remapping>/controller_manager:=controller_manager</remapping>
             </ros>
-            <parameters>$(find arm_gazebo)/params/arm_controllers.yaml</parameters>
         </plugin>
     </gazebo>

File: arm_description/urdf/camera.xacro (robot description, xacro)
@@ -3,5 +3,6 @@
   <link name='camera_link'>
     <visual>
-      <geometry><mesh filename="package://arm_description/meshes/camera.stl"/></geometry><material name="black"/>
+      <geometry><mesh filename="package://arm_description/meshes/camera.stl"/></geometry>
+      <material name="black"/>
     </visual>
     <collision>
@@ -31,13 +32,25 @@
   <gazebo reference="camera_optical_frame">
     <sensor type="camera" name="my_camera">
-      <topic>/camera/image_raw</topic>
+      <topic>camera/image_raw</topic>
       <update_rate>30.0</update_rate>
+      <visualize>true</visualize>
+      <always_on>1</always_on>
       <camera name="head">
+        <pose>0 0 0 0 0 0</pose>
         <horizontal_fov>1.0466</horizontal_fov>
-        <image><width>800</width><height>600</height><format>R8G8B8</format></image>
-        <clip><near>0.02</near><far>300</far></clip>
+        <image>
+          <width>800</width>
+          <height>600</height>
+          <format>R8G8B8</format>
+        </image>
+        <clip>
+          <near>0.02</near>
+          <far>300</far>
+        </clip>
         <distortion>
-          <k1>-0.414921465</k1><k2>0.277976117</k2>
-          <p1>0.000362302582</p1><p2>-0.000173492775</p2>
+          <k1>-0.414921465</k1>
+          <k2>0.277976117</k2>
+          <p1>0.000362302582</p1>
+          <p2>-0.000173492775</p2>
           <k3>-0.194112104</k3>
           <center>0.5 0.5</center>
